File: Hardware/Coaster.kicad_pcb (KiCad board)
At the start: 2 copper layers, 90 x 90 mm, 16 parts, among them J1 Conn_02x03_Odd_Even, U1 ATtiny85-20SU, U2 MAX619_MyOwn

Commit message: Changed LEDs to 5050 and switch to standard SPDT
Parts:
- D1, D2, D3, D4: footprint MyOwn:WS2812_2020_SMD -> LED_SMD:LED_WS2812B_PLCC4_5.0x5.0mm_P3.2mm
- S1: footprint MyOwn:Skjutomkopplare 1-pol on-on pcb vinklad -> Button_Switch_SMD:SW_SPDT_PCM12
- moved S1 9.22 mm to (68.5, 70.0), turned to 270 degrees
Routing:
- net 5V: track 239.2 -> 253.2 mm
- net 3V: track 51.8 -> 61.8 mm
- net GND: track 293.0 -> 302.2 mm
- net Net-(D2-Pad2): track 79.8 -> 71.5 mm
- net Net-(BT1-Pad1): track 163.6 -> 171.7 mm
- net Net-(D1-Pad2): track 71.5 -> 64.4 mm, vias 0 -> 2
- net Net-(D3-Pad2): track 62.8 -> 64.0 mm, vias 2 -> 0
- net MOSI: track 36.9 -> 37.9 mm
